Commit message: Temp fix for visuals of end effector

File: baxter_description/urdf/baxter_no_visual_grippers.urdf (robot description, URDF)
Before this commit: robot baxter, 49 links, 48 joints
Links:
- link left_gripper_l_finger: geometry collision box size=0.015 .1 .015; visual mesh filename=package://baxter_description/meshes/electric_gripper/finger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
- link left_gripper_r_finger: geometry collision box size=0.015 .1 .015; visual mesh filename=package://baxter_description/meshes/electric_gripper/finger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
- link right_gripper: geometry collision cylinder length=0.1 radius=0.0275
- link right_gripper_l_finger: geometry collision box size=0.015 .1 .015
- link right_gripper_r_finger: geometry collision box size=0.015 .1 .015
- link right_hand: geometry collision cylinder length=0.0464 radius=0.04; visual cylinder length=0.0464 radius=0.04
