Commit message: Syncing urdfs

File: baxter_description/urdf/hardware.baxter.urdf (robot description, URDF)
Before this commit: robot baxter, 49 links, 48 joints
Links:
- removed link left_gripper_l_finger
- removed link left_gripper_r_finger
- removed link right_gripper_l_finger
- removed link right_gripper_r_finger
- removed link screen_visual
- added link left_gripper_base, mass 0.0001; visual box size=0.025 0.075 0.035
- added link right_gripper_base, mass 0.0001; visual box size=0.025 0.075 0.035
- link base: mass None -> 0.0001
- link collision_head_link_1: mass 0.00094542 -> 0.0001
- link collision_head_link_2: mass 0.00094542 -> 0.0001
- link dummyhead1: mass 0.00094542 -> 0.0001
- link head_camera: mass 0.00094542 -> 0.0001
- link left_arm_itb: mass 0.00094542 -> 0.0001
- link left_arm_mount: mass 0.00094542 -> 0.0001
- link left_gripper: mass 0.00094542 -> 0.0001; geometry visual box size=0.01 0.01 0.01
- link left_hand_camera: mass 0.00094542 -> 0.0001
- link left_hand_camera_axis: mass 0.00094542 -> 0.0001
- link left_hand_range: mass 0.00094542 -> 0.0001
- link left_lower_elbow: geometry collision cylinder length=0.10 radius=0.06; visual mesh filename=package://baxter_description/meshes/lower_elbow/E1.DAE
- link left_torso_itb: mass 0.00094542 -> 0.0001
- link left_upper_elbow_visual: mass 0.00094542 -> 0.0001; geometry collision cylinder length=0.273 radius=0.06
- link left_upper_forearm_visual: mass 0.00094542 -> 0.0001; geometry collision cylinder length=0.272 radius=0.06
- link pedestal: geometry collision box size=0.92 0.83 0.3; visual mesh filename=package://baxter_description/meshes/base/PEDESTAL.DAE
- link right_arm_itb: mass 0.00094542 -> 0.0001
- link right_arm_mount: mass 0.00094542 -> 0.0001
- link right_gripper: mass 0.00094542 -> 0.0001; geometry visual box size=0.01 0.01 0.01
- link right_hand: geometry collision cylinder length=0.0464 radius=0.04
- link right_hand_camera: mass 0.00094542 -> 0.0001
- link right_hand_camera_axis: mass 0.00094542 -> 0.0001
- link right_hand_range: mass 0.00094542 -> 0.0001
- link right_lower_elbow: geometry collision cylinder length=0.10 radius=0.06; visual mesh filename=package://baxter_description/meshes/lower_elbow/E1.DAE
- link right_torso_itb: mass 0.00094542 -> 0.0001
- link right_upper_elbow_visual: mass 0.00094542 -> 0.0001; geometry collision cylinder length=0.273 radius=0.06
- link right_upper_forearm_visual: mass 0.00094542 -> 0.0001; geometry collision cylinder length=0.272 radius=0.06
- link sonar_ring: mass 0.00094542 -> 0.0001
- link torso: geometry collision cylinder length=0.7 radius=0.27; visual mesh filename=package://baxter_description/meshes/torso/base_link.DAE
Joints:
- removed joint left_gripper_l_finger_joint
- removed joint left_gripper_r_finger_joint
- removed joint right_gripper_l_finger_joint
- removed joint right_gripper_r_finger_joint
- removed joint screen_visual_joint
- added joint left_gripper_base: type fixed, parent left_hand, child left_gripper_base, origin xyz=0 0 0 rpy=0 0 0
- added joint right_gripper_base: type fixed, parent right_hand, child right_gripper_base, origin xyz=0 0 0 rpy=0 0 0
- joint head_camera: origin xyz=0.12839 0.0 0.06368 rpy=0.0 0.61073254 0.0 -> xyz=0.12839 0 0.06368 rpy=1.75057 0 1.57079632679
- joint head_nod: origin xyz=.088 0.0 0.0 rpy=1.9198622 0.0 1.57079632679 -> xyz=.1227 0 0 rpy=1.75057 0 1.57079632679
- joint head_pan: origin xyz=0.0947 0 0.686 rpy=0 0 0 -> xyz=0.06 0 0.686 rpy=0 0 0
- joint left_e0: limit lower=-3.05417993878 upper=3.05417993878 effort=60.0 velocity=2.5 -> lower=-3.05417993878 upper=3.05417993878 effort=50.0 velocity=1.5
- joint left_e1: limit lower=-0.05 upper=2.618 effort=60.0 velocity=2.5 -> lower=-0.05 upper=2.618 effort=50.0 velocity=1.5
- joint left_endpoint: origin xyz=-0.005 0.0 0.02 rpy=1.57 0 0 -> xyz=0.0 0 0.025 rpy=0 0 0; parent left_hand -> left_gripper_base
- joint left_hand_camera: origin xyz=0.03825 0.012 0.015355 rpy=0 -1.57079633 0 -> xyz=0.03825 0.012 0.015355 rpy=0 0 -1.57079633
- joint left_s0: limit lower=-1.70167993878 upper=1.70167993878 effort=60.0 velocity=2.5 -> lower=-1.70167993878 upper=1.70167993878 effort=50.0 velocity=1.5
- joint left_s1: limit lower=-2.147 upper=1.047 effort=60.0 velocity=2.5 -> lower=-2.147 upper=1.047 effort=50.0 velocity=1.5
- joint left_w0: limit lower=-3.059 upper=3.059 effort=20.0 velocity=5.0 -> lower=-3.059 upper=3.059 effort=15.0 velocity=4.0
- joint left_w1: limit lower=-1.57079632679 upper=2.094 effort=20.0 velocity=5.0 -> lower=-1.57079632679 upper=2.094 effort=15.0 velocity=4.0
- joint left_w2: limit lower=-3.059 upper=3.059 effort=20.0 velocity=5.0 -> lower=-3.059 upper=3.059 effort=15.0 velocity=4.0
- joint right_e0: limit lower=-3.05417993878 upper=3.05417993878 effort=60.0 velocity=2.5 -> lower=-3.05417993878 upper=3.05417993878 effort=50.0 velocity=1.5
- joint right_e1: limit lower=-0.05 upper=2.618 effort=60.0 velocity=2.5 -> lower=-0.05 upper=2.618 effort=50.0 velocity=1.5
- joint right_endpoint: origin xyz=-0.005 0.0 0.02 rpy=1.57 0 0 -> xyz=0.0 0 0.025 rpy=0 0 0; parent right_hand -> right_gripper_base
- joint right_hand_camera: origin xyz=0.03825 0.012 0.015355 rpy=0 -1.57079633 0 -> xyz=0.03825 0.012 0.015355 rpy=0 0 -1.57079633
- joint right_s0: limit lower=-1.70167993878 upper=1.70167993878 effort=60.0 velocity=2.5 -> lower=-1.70167993878 upper=1.70167993878 effort=50.0 velocity=1.5
- joint right_s1: limit lower=-2.147 upper=1.047 effort=60.0 velocity=2.5 -> lower=-2.147 upper=1.047 effort=50.0 velocity=1.5
- joint right_w0: limit lower=-3.059 upper=3.059 effort=20.0 velocity=5.0 -> lower=-3.059 upper=3.059 effort=15.0 velocity=4.0
- joint right_w1: limit lower=-1.57079632679 upper=2.094 effort=20.0 velocity=5.0 -> lower=-1.57079632679 upper=2.094 effort=15.0 velocity=4.0
- joint right_w2: limit lower=-3.059 upper=3.059 effort=20.0 velocity=5.0 -> lower=-3.059 upper=3.059 effort=15.0 velocity=4.0
