Commit message: Resynced custom URDF with URDF shipped on Baxter

File: baxter_description/urdf/my_old_custom.baxter.urdf (robot description, URDF)
Before this commit: robot baxter, 50 links, 49 joints
Links:
- removed link left_gripper_base
- removed link right_gripper_base
- removed link right_gripper_l_finger
- removed link right_gripper_r_finger
- added link screen_visual, mass 0.001; visual box size=0.218 0.16 0.001
- link collision_head_link_1: mass 0.0001 -> 0.00094542
- link collision_head_link_2: mass 0.0001 -> 0.00094542
- link dummyhead1: mass 0.0001 -> 0.00094542
- link head_camera: mass 0.0001 -> 0.00094542
- link left_arm_itb: mass 0.0001 -> 0.00094542
- link left_arm_mount: mass 0.0001 -> 0.00094542
- link left_hand_camera: mass 0.0001 -> 0.00094542
- link left_hand_camera_axis: mass 0.0001 -> 0.00094542
- link left_hand_range: mass 0.0001 -> 0.00094542
- link left_lower_elbow: geometry collision cylinder length=0.18 radius=0.076; visual mesh filename=package://baxter_description/meshes/lower_elbow/E1.DAE
- link left_upper_elbow_visual: mass 0.0001 -> 0.00094542; geometry collision cylinder length=0.30 radius=0.084
- link left_upper_forearm_visual: mass 0.0001 -> 0.00094542; geometry collision cylinder length=0.272 radius=0.068
- link pedestal: geometry collision box size=0.9 0.9 0.3; collision cylinder length=0.6 radius=0.15
- link right_arm_itb: mass 0.0001 -> 0.00094542
- link right_arm_mount: mass 0.0001 -> 0.00094542
- link right_hand: geometry 
- link right_hand_camera: mass 0.0001 -> 0.00094542
- link right_hand_camera_axis: mass 0.0001 -> 0.00094542
- link right_hand_range: mass 0.0001 -> 0.00094542
- link right_lower_elbow: geometry collision cylinder length=0.18 radius=0.076; visual mesh filename=package://baxter_description/meshes/lower_elbow/E1.DAE
- link right_upper_elbow_visual: mass 0.0001 -> 0.00094542; geometry collision cylinder length=0.30 radius=0.084
- link right_upper_forearm_visual: mass 0.0001 -> 0.00094542; geometry collision cylinder length=0.272 radius=0.068
- link sonar_ring: mass 0.0001 -> 0.00094542
- link torso: geometry collision mesh filename=package://baxter_description/meshes/torso/base_link_simple.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; visual mesh filename=package://baxter_description/meshes/torso/base_link.DAE
Joints:
- removed joint left_gripper_base
- removed joint right_gripper_base
- removed joint right_gripper_l_finger_joint
- removed joint right_gripper_r_finger_joint
- added joint screen_visual_joint: type fixed, parent screen, child screen_visual, origin xyz=0.0 -0.016 0.0 rpy=0 0 0
- joint head_camera: origin xyz=0.12839 0 0.06368 rpy=1.75057 0 1.57079632679 -> xyz=0.12839 0.0 0.06368 rpy=0.0 0.61073254 0.0
- joint head_nod: origin xyz=.1227 0 0 rpy=1.75057 0 1.57079632679 -> xyz=.088 0.0 0.0 rpy=1.9198622 0.0 1.57079632679
- joint head_pan: origin xyz=0.06 0 0.686 rpy=0 0 0 -> xyz=0.0947 0 0.686 rpy=0 0 0
- joint left_e0: limit lower=-3.05417993878 upper=3.05417993878 effort=50.0 velocity=1.5 -> lower=-3.05417993878 upper=3.05417993878 effort=60.0 velocity=2.5
- joint left_e1: limit lower=-0.05 upper=2.618 effort=50.0 velocity=1.5 -> lower=-0.05 upper=2.618 effort=60.0 velocity=2.5
- joint left_endpoint: origin xyz=0.0 0 0.025 rpy=0 0 0 -> xyz=-0.005 0.0 0.02 rpy=1.57 0 0; parent left_gripper_base -> left_hand
- joint left_gripper_l_finger_joint: axis 0 1 0 -> 0 0 1
- joint left_gripper_r_finger_joint: axis 0 1 0 -> 0 0 1; origin xyz=0.0 0.06 0.035 rpy=0 0 0 -> xyz=0.0 0.06 -0.035 rpy=0 0 0
- joint left_hand_camera: origin xyz=0.03825 0.012 0.015355 rpy=0 0 -1.57079633 -> xyz=0.03825 0.012 0.015355 rpy=0 -1.57079633 0
- joint left_s0: limit lower=-1.70167993878 upper=1.70167993878 effort=50.0 velocity=1.5 -> lower=-1.70167993878 upper=1.70167993878 effort=60.0 velocity=2.5
- joint left_s1: limit lower=-2.147 upper=1.047 effort=50.0 velocity=1.5 -> lower=-2.147 upper=1.047 effort=60.0 velocity=2.5
- joint left_w0: limit lower=-3.059 upper=3.059 effort=15.0 velocity=4.0 -> lower=-3.059 upper=3.059 effort=20.0 velocity=5.0
- joint left_w1: limit lower=-1.57079632679 upper=2.094 effort=15.0 velocity=4.0 -> lower=-1.57079632679 upper=2.094 effort=20.0 velocity=5.0
- joint left_w2: limit lower=-3.059 upper=3.059 effort=15.0 velocity=4.0 -> lower=-3.059 upper=3.059 effort=20.0 velocity=5.0
- joint right_e0: limit lower=-3.05417993878 upper=3.05417993878 effort=50.0 velocity=1.5 -> lower=-3.05417993878 upper=3.05417993878 effort=60.0 velocity=2.5
- joint right_e1: limit lower=-0.05 upper=2.618 effort=50.0 velocity=1.5 -> lower=-0.05 upper=2.618 effort=60.0 velocity=2.5
- joint right_endpoint: origin xyz=0.0 0 0.025 rpy=0 0 0 -> xyz=-0.005 0.0 0.02 rpy=1.57 0 0; parent right_gripper_base -> right_hand
- joint right_hand_camera: origin xyz=0.03825 0.012 0.015355 rpy=0 0 -1.57079633 -> xyz=0.03825 0.012 0.015355 rpy=0 -1.57079633 0
- joint right_s0: limit lower=-1.70167993878 upper=1.70167993878 effort=50.0 velocity=1.5 -> lower=-1.70167993878 upper=1.70167993878 effort=60.0 velocity=2.5
- joint right_s1: limit lower=-2.147 upper=1.047 effort=50.0 velocity=1.5 -> lower=-2.147 upper=1.047 effort=60.0 velocity=2.5
- joint right_w0: limit lower=-3.059 upper=3.059 effort=15.0 velocity=4.0 -> lower=-3.059 upper=3.059 effort=20.0 velocity=5.0
- joint right_w1: limit lower=-1.57079632679 upper=2.094 effort=15.0 velocity=4.0 -> lower=-1.57079632679 upper=2.094 effort=20.0 velocity=5.0
- joint right_w2: limit lower=-3.059 upper=3.059 effort=15.0 velocity=4.0 -> lower=-3.059 upper=3.059 effort=20.0 velocity=5.0
