Commit message: renamed old baxter.urdf, replaced with open hand urdf.

File: baxter_description/urdf/baxter_dual_electric_grippers.urdf (robot description, URDF)
Before this commit: robot baxter, 53 links, 52 joints
Links:
- link left_gripper_base: geometry collision cylinder length=0.1 radius=0.0275; visual mesh filename=package://baxter_description/meshes/electric_gripper/electr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 scale=1 1 1
- link left_gripper_l_finger: geometry collision cylinder length=0.115 radius=0.008; visual mesh filename=package://baxter_description/meshes/electric_gripper/finger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
- link left_gripper_r_finger: geometry collision cylinder length=0.115 radius=0.01; visual mesh filename=package://baxter_description/meshes/electric_gripper/finger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
- link right_gripper_base: geometry collision cylinder length=0.1 radius=0.0275; visual mesh filename=package://baxter_description/meshes/electric_gripper/electr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 scale=1 1 1
- link right_gripper_l_finger: geometry collision cylinder length=0.115 radius=0.008; visual mesh filename=package://baxter_description/meshes/electric_gripper/finger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
- link right_gripper_r_finger: geometry collision cylinder length=0.115 radius=0.01; visual mesh filename=package://baxter_description/meshes/electric_gripper/finger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
Joints:
- joint left_gripper_l_finger_joint: limit lower=-1.5708 upper=0 effort=20.0 velocity=5.0 -> lower=-0.0125 upper=0.0095 effort=20.0 velocity=5.0; origin xyz=0.01833 -0.024 0.074 rpy=0 -1.5708 0 -> xyz=0.0 -0.04 0.035 rpy=1.57 0 0; type revolute -> prismatic
- joint left_gripper_r_finger_joint: limit lower=0 upper=1.5708 effort=20.0 velocity=5.0 -> lower=-0.0125 upper=0.0095 effort=20.0 velocity=5.0; mimic joint=left_gripper_l_finger_joint multiplier=1 offset=0 -> joint=left_gripper_l_finger_joint multiplier=-1 offset=0; origin xyz=-0.01833 0.019 0.074 rpy=0 -1.5708 3.14159 -> xyz=0.0 0.04 0.035 rpy=1.57 0 0; type revolute -> prismatic
- joint right_gripper_l_finger_joint: limit lower=-1.5708 upper=0 effort=20.0 velocity=5.0 -> lower=-0.0125 upper=0.0095 effort=20.0 velocity=5.0; origin xyz=0.01833 -0.024 0.074 rpy=0 -1.5708 0 -> xyz=0.0 -0.04 0.035 rpy=1.57 0 0; type revolute -> prismatic
- joint right_gripper_r_finger_joint: limit lower=0 upper=1.5708 effort=20.0 velocity=5.0 -> lower=-0.0125 upper=0.0095 effort=20.0 velocity=5.0; mimic joint=right_gripper_l_finger_joint multiplier=1 offset=0 -> joint=right_gripper_l_finger_joint multiplier=-1 offset=0; origin xyz=-0.01833 0.019 0.074 rpy=0 -1.5708 3.14159 -> xyz=0.0 0.04 0.035 rpy=1.57 0 0; type revolute -> prismatic
