Commit message: finished urdf and added color to model

File: baxter_description/urdf/baxter_open_hand.urdf (robot description, URDF)
Before this commit: robot baxter, 55 links, 54 joints
Links:
- added link right_gripper_l_second_finger, mass 0.00094542; collision mesh filename=package://baxter_description/meshes/open_hand_gripper/finge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 scale=0.01 0.01 0.01; visual mesh filename=package://baxter_description/meshes/open_hand_gripper/finge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 scale=0.01 0.01 0.01
- added link right_gripper_r_second_finger, mass 0.00094542; collision mesh filename=package://baxter_description/meshes/open_hand_gripper/finge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 scale=0.01 0.01 0.01; visual mesh filename=package://baxter_description/meshes/open_hand_gripper/finge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 scale=0.01 0.01 0.01
- link left_gripper_base: geometry collision mesh filename=package://baxter_description/meshes/open_hand_gripper/base.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 scale=0.01 0.01 0.01; visual mesh filename=package://baxter_description/meshes/open_hand_gripper/base.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 scale=0.01 0.01 0.01
- link left_gripper_l_finger: geometry collision mesh filename=package://baxter_description/meshes/open_hand_gripper/finge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 scale=0.01 0.01 0.01; visual mesh filename=package://baxter_description/meshes/open_hand_gripper/finge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 scale=0.01 0.01 0.01
- link left_gripper_l_second_finger: geometry collision mesh filename=package://baxter_description/meshes/open_hand_gripper/finge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 scale=0.01 0.01 0.01; visual mesh filename=package://baxter_description/meshes/open_hand_gripper/finge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 scale=0.01 0.01 0.01
- link left_gripper_r_finger: geometry collision mesh filename=package://baxter_description/meshes/open_hand_gripper/finge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 scale=0.01 0.01 0.01; visual mesh filename=package://baxter_description/meshes/open_hand_gripper/finge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 scale=0.01 0.01 0.01
- link left_gripper_r_second_finger: geometry collision mesh filename=package://baxter_description/meshes/open_hand_gripper/finge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 scale=0.01 0.01 0.01; visual mesh filename=package://baxter_description/meshes/open_hand_gripper/finge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 scale=0.01 0.01 0.01
- link right_gripper_base: geometry collision mesh filename=package://baxter_description/meshes/open_hand_gripper/base.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 scale=0.01 0.01 0.01; visual mesh filename=package://baxter_description/meshes/open_hand_gripper/base.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 scale=0.01 0.01 0.01
- link right_gripper_l_finger: geometry collision mesh filename=package://baxter_description/meshes/open_hand_gripper/finge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 scale=0.01 0.01 0.01; visual mesh filename=package://baxter_description/meshes/open_hand_gripper/finge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 scale=0.01 0.01 0.01
- link right_gripper_r_finger: geometry collision mesh filename=package://baxter_description/meshes/open_hand_gripper/finge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 scale=0.01 0.01 0.01; visual mesh filename=package://baxter_description/meshes/open_hand_gripper/finge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 scale=0.01 0.01 0.01
Joints:
- added joint right_gripper_l_second_finger_joint: type revolute, parent right_gripper, child right_gripper_l_second_finger, origin xyz=0.017165 -0.024 0.074 rpy=0 -1.5708 0, axis 0 0 1, limit lower=-1.5708 upper=0 effort=20.0 velocity=5.0, mimic joint=right_gripper_l_finger_joint multiplier=1 offset=0
- added joint right_gripper_r_second_finger_joint: type revolute, parent right_gripper, child right_gripper_r_second_finger, origin xyz=0.019495 0.024 0.074 rpy=0 -1.5708 3.14159, axis 0 0 1, limit lower=0.0 upper=1.5708 effort=20.0 velocity=5.0, mimic joint=right_gripper_l_finger_joint multiplier=1 offset=0
- joint right_gripper_l_finger_joint: limit lower=-0.0125 upper=0.0095 effort=20.0 velocity=5.0 -> lower=-1.5708 upper=0 effort=20.0 velocity=5.0; origin xyz=0.0 -0.04 0.035 rpy=1.57 0 0 -> xyz=-0.019495 -0.024 0.074 rpy=0 -1.5708 0; type prismatic -> revolute
- joint right_gripper_r_finger_joint: limit lower=-0.0125 upper=0.0095 effort=20.0 velocity=5.0 -> lower=0 upper=1.5708 effort=20.0 velocity=5.0; mimic joint=right_gripper_l_finger_joint multiplier=-1 offset=0 -> joint=right_gripper_l_finger_joint multiplier=1 offset=0; origin xyz=0.0 0.04 0.035 rpy=1.57 0 0 -> xyz=-0.017165 0.024 0.074 rpy=0 -1.5708 3.14159; type prismatic -> revolute

Commit message: updated urdf

File: baxter_description/urdf/baxter_open_hand.urdf (robot description, URDF)
Before this commit: robot baxter, 57 links, 56 joints
Links:
- removed link left_gripper_l_second_finger
- removed link left_gripper_r_second_finger
- removed link right_gripper_l_second_finger
- removed link right_gripper_r_second_finger
Joints:
- removed joint left_gripper_l_second_finger_joint
- removed joint left_gripper_r_second_finger_joint
- removed joint right_gripper_l_second_finger_joint
- removed joint right_gripper_r_second_finger_joint
- joint left_gripper_l_finger_joint: origin xyz=-0.019495 -0.024 0.074 rpy=0 -1.5708 0 -> xyz=0.01833 -0.024 0.074 rpy=0 -1.5708 0
- joint left_gripper_r_finger_joint: origin xyz=-0.017165 0.024 0.074 rpy=0 -1.5708 3.14159 -> xyz=-0.01833 0.019 0.074 rpy=0 -1.5708 3.14159
- joint right_gripper_l_finger_joint: origin xyz=-0.019495 -0.024 0.074 rpy=0 -1.5708 0 -> xyz=0.01833 -0.024 0.074 rpy=0 -1.5708 0
- joint right_gripper_r_finger_joint: origin xyz=-0.017165 0.024 0.074 rpy=0 -1.5708 3.14159 -> xyz=-0.01833 0.019 0.074 rpy=0 -1.5708 3.14159

Commit message: yale open hands are now open at 0.0 and closed at 1.5708

File: baxter_description/urdf/baxter_open_hand.urdf (robot description, URDF)
Before this commit: robot baxter, 53 links, 52 joints
Joints:
- joint left_gripper_l_finger_joint: limit lower=-1.5708 upper=0 effort=20.0 velocity=5.0 -> lower=0 upper=1.5708 effort=20.0 velocity=5.0
- joint right_gripper_l_finger_joint: limit lower=-1.5708 upper=0 effort=20.0 velocity=5.0 -> lower=0 upper=1.5708 effort=20.0 velocity=5.0
