Commit message: Added tip link to end effector Removed "trash" folder

File: baxter_description/urdf/baxter.urdf.xacro (robot description, xacro)
@@ -6,5 +6,5 @@
        xmlns:xi="http://www.w3.org/2001/XInclude">
 <xacro:include filename="$(find baxter_description)/urdf/baxter_no_end_effectors.urdf"/>
-<xacro:include filename="$(find baxter_description)/urdf/open_hand.urdf.xacro" />
+<!-- <xacro:include filename="$(find baxter_description)/urdf/open_hand.urdf.xacro" /> -->
 <xacro:include filename="$(find baxter_description)/urdf/electric_gripper.urdf.xacro" />
 <!-- Electric Parallel Gripper -->

File: baxter_description/urdf/baxter_no_end_effectors.urdf (robot description, URDF)
Before this commit: robot None, 47 links, 46 joints
Links:
- added link left_gripper_tip
- added link right_gripper_tip

File: baxter_description/urdf/electric_gripper.urdf.xacro (robot description, xacro)
@@ -73,5 +73,5 @@
     </collision>
   </link>
-  <!-- Base of Left end effector -->
+  <!-- Base of end effector -->
   <joint name="${arm}_endpoint" type="fixed">
     <origin xyz="0 0 0.045" rpy="0 -0 0" />
@@ -99,4 +99,11 @@
     <mimic joint="${arm}_gripper_l_finger_joint" offset="0" multiplier="-1" />
   </joint>
+  <!-- Tip of end effector -->
+  <joint name="${arm}_endpoint2" type="fixed">
+    <origin xyz="0 0 0.115" rpy="0 -0 0" />
+    <axis xyz="0 0 0" />
+    <parent link="${arm}_gripper" />
+    <child link="${arm}_gripper_tip" />
+  </joint>
 </xacro:macro>
 </robot>
