Commit message: Make arms welded onto frame exactly the same (breaks calibration)

File: baxter_description/urdf/baxter_no_end_effectors.urdf (robot description, URDF)
Before this commit: robot None, 49 links, 46 joints
Joints:
- joint left_torso_arm_mount: origin xyz=0.0252503 0.219489 0.109759 rpy=-0.00479639 0.00185872 0.779972 -> xyz=0.023277  0.21986  0.10804 rpy=-0.0174986  0.00342261 0.785584
