Commit message: Change gripper joint name to reflect Baxter 1.2 API name change

File: baxter_description/urdf/electric_gripper.urdf.xacro (robot description, xacro)
@@ -81,5 +81,11 @@
   </joint>
   <!-- Left finger -->
-  <joint name="${arm}_gripper_l_finger_joint" type="prismatic">
+  <xacro:if value="${arm == 'right'}">
+    <xacro:property name="arm_short" value="r" />
+  </xacro:if>
+  <xacro:if value="${arm == 'left'}">
+    <xacro:property name="arm_short" value="l" />
+  </xacro:if>
+  <joint name="${arm_short}_gripper_l_finger_joint" type="prismatic">
     <origin rpy="1.57 0 0" xyz="0.0 -0.04 0.035"/>
     <axis xyz="0 0 1"/>
@@ -97,5 +103,5 @@
     <limit effort="20.0" lower="-0.0125" upper="0.0095" velocity="5.0"/> <!-- upper is open -->
     <dynamics damping="0.7" friction="0.0"/>
-    <mimic joint="${arm}_gripper_l_finger_joint" offset="0" multiplier="-1" />
+    <mimic joint="${arm_short}_gripper_l_finger_joint" offset="0" multiplier="-1" />
   </joint>
   <!-- Tip of end effector -->

Commit message: Move fingers together to simulate holding dry erase markers for whiteboard

File: baxter_description/urdf/electric_gripper.urdf.xacro (robot description, xacro)
@@ -7,5 +7,5 @@
   <link name="${arm}_gripper_l_finger">
     <visual>
-      <origin rpy="0 -1.57079632679 0" xyz="0.0 -0.036 -0.0135"/>
+      <origin rpy="0 -1.57079632679 0" xyz="0.0 -0.036 -0.05"/>
       <geometry>
         <mesh filename="package://baxter_description/meshes/electric_gripper/fingers/extended_narrow.DAE" /> <!-- Long left finger-->
@@ -16,5 +16,5 @@
     </visual>
     <collision>
-      <origin rpy="1.57 0 0" xyz="0.00 0.02 0.005" />
+      <origin rpy="1.57 0 0" xyz="0.00 0.02 -0.045" />
       <geometry>
 	<cylinder length="0.115" radius="0.008" />
@@ -30,5 +30,5 @@
   <link name="${arm}_gripper_r_finger">
     <visual>
-      <origin rpy="0 1.57079632679 0" xyz="0.0 -0.036 0.0135"/>
+      <origin rpy="0 1.57079632679 0" xyz="0.0 -0.036 0.05"/>
       <geometry>
         <mesh filename="package://baxter_description/meshes/electric_gripper/fingers/extended_narrow.DAE" /> <!-- Long left finger-->
@@ -39,5 +39,5 @@
     </visual>
     <collision>
-      <origin rpy="1.57 0 0" xyz="0.00 0.02 -0.005" />
+      <origin rpy="1.57 0 0" xyz="0.00 0.02 0.045" />
       <geometry>
 	<cylinder length="0.115" radius="0.01" />
