Commit message: Increased collision sizes, fixed fingers, changed torso mesh

File: baxter_description/urdf/baxter.urdf (robot description, URDF)
Before this commit: robot baxter, 53 links, 52 joints
Links:
- link left_gripper: geometry collision cylinder length=0.1 radius=0.0275; visual box size=0.01 0.01 0.01
- link left_gripper_l_finger: geometry collision cylinder length=0.115 radius=0.008; visual mesh filename=package://baxter_description/meshes/electric_gripper/finger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
- link left_gripper_r_finger: geometry collision cylinder length=0.115 radius=0.01; visual mesh filename=package://baxter_description/meshes/electric_gripper/finger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
- link left_lower_elbow: geometry collision cylinder length=0.1 radius=0.07; visual mesh filename=package://baxter_description/meshes/lower_elbow/E1.DAE scale=1 1 1
- link left_lower_forearm: geometry collision cylinder length=0.1 radius=0.07; visual mesh filename=package://baxter_description/meshes/lower_forearm/W1.DAE scale=1 1 1
- link left_lower_shoulder: geometry collision cylinder length=0.12 radius=0.07; visual mesh filename=package://baxter_description/meshes/lower_shoulder/S1.DAE scale=1 1 1
- link left_upper_elbow: geometry collision cylinder length=0.107 radius=0.07; visual mesh filename=package://baxter_description/meshes/upper_elbow/E0.DAE scale=1 1 1
- link left_upper_elbow_visual: geometry collision cylinder length=0.273 radius=0.08
- link left_upper_forearm: geometry collision cylinder length=0.088 radius=0.07; visual mesh filename=package://baxter_description/meshes/upper_forearm/W0.DAE scale=1 1 1
- link left_upper_forearm_visual: geometry collision cylinder length=0.272 radius=0.07
- link left_upper_shoulder: geometry collision cylinder length=0.2722 radius=0.07; visual mesh filename=package://baxter_description/meshes/upper_shoulder/S0.DAE scale=1 1 1
- link pedestal: geometry collision cylinder length=0.6 radius=0.15; visual mesh filename=package://baxter_description/meshes/base/PEDESTAL.DAE scale=1 1 1
- link right_gripper: geometry collision cylinder length=0.1 radius=0.0275; visual box size=0.01 0.01 0.01
- link right_gripper_l_finger: geometry collision cylinder length=0.115 radius=0.008; visual mesh filename=package://baxter_description/meshes/electric_gripper/finger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
- link right_gripper_r_finger: geometry collision cylinder length=0.115 radius=0.01; visual mesh filename=package://baxter_description/meshes/electric_gripper/finger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
- link right_lower_elbow: geometry collision cylinder length=0.1 radius=0.07; visual mesh filename=package://baxter_description/meshes/lower_elbow/E1.DAE scale=1 1 1
- link right_lower_forearm: geometry collision cylinder length=0.1 radius=0.07; visual mesh filename=package://baxter_description/meshes/lower_forearm/W1.DAE scale=1 1 1
- link right_lower_shoulder: geometry collision cylinder length=0.12 radius=0.07; visual mesh filename=package://baxter_description/meshes/lower_shoulder/S1.DAE scale=1 1 1
- link right_upper_elbow: geometry collision cylinder length=0.107 radius=0.07; visual mesh filename=package://baxter_description/meshes/upper_elbow/E0.DAE scale=1 1 1
- link right_upper_elbow_visual: geometry collision cylinder length=0.273 radius=0.08
- link right_upper_forearm: geometry collision cylinder length=0.088 radius=0.07; visual mesh filename=package://baxter_description/meshes/upper_forearm/W0.DAE scale=1 1 1
- link right_upper_forearm_visual: geometry collision cylinder length=0.272 radius=0.07
- link right_upper_shoulder: geometry collision cylinder length=0.2722 radius=0.07; visual mesh filename=package://baxter_description/meshes/upper_shoulder/S0.DAE scale=1 1 1
- link torso: geometry collision mesh filename=package://baxter_description/meshes/torso/base_link_simple.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; visual mesh filename=package://baxter_description/meshes/torso/base_link.DAE scale=1 1 1

Commit message: Tweaked URDF for bigger collision model

File: baxter_description/urdf/baxter.urdf (robot description, URDF)
Before this commit: robot baxter, 53 links, 52 joints
Links:
- link collision_head_link_1: geometry collision sphere radius=0.25; visual sphere radius=0.001
- link collision_head_link_2: geometry collision sphere radius=0.25; visual sphere radius=0.001
- link left_upper_elbow_visual: geometry collision cylinder length=0.28 radius=0.082

Commit message: Added better collision meshes for grippers

File: baxter_description/urdf/baxter.urdf (robot description, URDF)
Before this commit: robot baxter, 53 links, 52 joints
Links:
- link left_gripper: geometry visual box size=0.01 0.01 0.01
- link left_gripper_base: geometry collision cylinder length=0.1 radius=0.0275; visual mesh filename=package://baxter_description/meshes/electric_gripper/electr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 scale=1 1 1
- link right_gripper: geometry visual box size=0.01 0.01 0.01
- link right_gripper_base: geometry collision cylinder length=0.1 radius=0.0275; visual mesh filename=package://baxter_description/meshes/electric_gripper/electr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 scale=1 1 1

Commit message: Increased size of collision shapes

File: baxter_description/urdf/baxter.urdf (robot description, URDF)
Before this commit: robot baxter, 53 links, 52 joints
Links:
- link left_lower_elbow: geometry collision cylinder length=0.18 radius=0.08; visual mesh filename=package://baxter_description/meshes/lower_elbow/E1.DAE scale=1 1 1
- link left_lower_forearm: geometry collision cylinder length=0.16 radius=0.06; visual mesh filename=package://baxter_description/meshes/lower_forearm/W1.DAE scale=1 1 1
- link left_lower_shoulder: geometry collision cylinder length=0.25 radius=0.09; visual mesh filename=package://baxter_description/meshes/lower_shoulder/S1.DAE scale=1 1 1
- link left_upper_elbow: geometry collision cylinder length=0.107 radius=0.09; visual mesh filename=package://baxter_description/meshes/upper_elbow/E0.DAE scale=1 1 1
- link left_upper_elbow_visual: geometry collision cylinder length=0.3 radius=0.09
- link left_upper_shoulder: geometry collision cylinder length=0.35 radius=0.1; visual mesh filename=package://baxter_description/meshes/upper_shoulder/S0.DAE scale=1 1 1
- link pedestal: geometry collision box size=0.8 0.8 0.25; collision cylinder length=0.11 radius=0.19
- link right_lower_elbow: geometry collision cylinder length=0.18 radius=0.08; visual mesh filename=package://baxter_description/meshes/lower_elbow/E1.DAE scale=1 1 1
- link right_lower_forearm: geometry collision cylinder length=0.16 radius=0.06; visual mesh filename=package://baxter_description/meshes/lower_forearm/W1.DAE scale=1 1 1
- link right_lower_shoulder: geometry collision cylinder length=0.25 radius=0.09; visual mesh filename=package://baxter_description/meshes/lower_shoulder/S1.DAE scale=1 1 1
- link right_upper_elbow: geometry collision cylinder length=0.107 radius=0.09; visual mesh filename=package://baxter_description/meshes/upper_elbow/E0.DAE scale=1 1 1
- link right_upper_elbow_visual: geometry collision cylinder length=0.3 radius=0.09
- link right_upper_shoulder: geometry collision cylinder length=0.35 radius=0.1; visual mesh filename=package://baxter_description/meshes/upper_shoulder/S0.DAE scale=1 1 1

Commit message: Small tweaks

File: baxter_description/urdf/baxter.urdf (robot description, URDF)
Before this commit: robot baxter, 53 links, 52 joints
Links:
- link pedestal: geometry collision cylinder length=0.6 radius=0.15; visual mesh filename=package://baxter_description/meshes/base/PEDESTAL.DAE scale=1 1 1

Commit message: Enabled collision Added script for viewing pdf Updated gitignore

File: baxter_description/urdf/baxter.urdf (robot description, URDF)
Before this commit: robot baxter, 53 links, 52 joints
Links:
- link pedestal: geometry collision box size=0.8 0.8 0.25; collision cylinder length=0.11 radius=0.19

Commit message: Increased pedestal size

File: baxter_description/urdf/baxter.urdf (robot description, URDF)
Before this commit: robot baxter, 53 links, 52 joints
Links:
- link pedestal: geometry collision box size=0.82 0.83 0.28; collision cylinder length=0.11 radius=0.19

Commit message: Disabled unnecessary links

File: baxter_description/urdf/baxter.urdf (robot description, URDF)
Before this commit: robot baxter, 53 links, 52 joints
Links:
- link left_hand_accelerometer: geometry 
- link right_hand_accelerometer: geometry 

Commit message: Reduced collision head size Changed Yale hand base to be primitive cylinder

File: baxter_description/urdf/baxter.urdf (robot description, URDF)
Before this commit: robot baxter, 53 links, 52 joints
Links:
- link collision_head_link_1: geometry collision sphere radius=0.18; visual sphere radius=0.001
- link collision_head_link_2: geometry collision sphere radius=0.18; visual sphere radius=0.001
- link right_gripper_base: geometry collision cylinder length=0.07 radius=0.05; visual mesh filename=package://baxter_description/meshes/open_hand_gripper/base.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 scale=0.01 0.01 0.01

Commit message: change to xacro for baxter urdf, moved extraneous files to trash folder

File: baxter_description/urdf/baxter.urdf (robot description, URDF)
Before this commit: robot baxter, 53 links, 52 joints
Links:
- link collision_head_link_1: geometry collision sphere radius=0.18; visual sphere radius=0.001
- link collision_head_link_2: geometry collision sphere radius=0.18; visual sphere radius=0.001
- link pedestal: geometry collision box size=0.2 0.325 0.28; collision box size=0.2 0.325 0.28
- link right_gripper_base: geometry collision cylinder length=0.08 radius=0.05; visual mesh filename=package://baxter_description/meshes/open_hand_gripper/base.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 scale=0.01 0.01 0.01
- link right_gripper_l_finger: geometry collision box size=0.021 0.036 0.055; collision box size=0.021 0.060 0.055
- link right_gripper_r_finger: geometry collision box size=0.021 0.036 0.055; collision box size=0.021 0.060 0.055
Joints:
- joint right_gripper_l_finger_joint: limit lower=-1.5708 upper=0 effort=20.0 velocity=5.0 -> lower=0 upper=1.5708 effort=20.0 velocity=5.0

File: baxter_description/urdf/baxter_no_end_effectors.urdf (robot description, URDF)
Before this commit: robot baxter, 53 links, 52 joints
Links:
- removed link left_gripper_base
- removed link left_gripper_l_finger
- removed link left_gripper_r_finger
- removed link right_gripper_base
- removed link right_gripper_l_finger
- removed link right_gripper_r_finger
- link collision_head_link_1: geometry collision sphere radius=0.18; visual sphere radius=0.001
- link collision_head_link_2: geometry collision sphere radius=0.18; visual sphere radius=0.001
- link pedestal: geometry collision box size=0.2 0.325 0.28; collision box size=0.2 0.325 0.28
Joints:
- removed joint left_endpoint
- removed joint left_gripper_l_finger_joint
- removed joint left_gripper_r_finger_joint
- removed joint right_endpoint
- removed joint right_gripper_l_finger_joint
- removed joint right_gripper_r_finger_joint
