Commit message: Reduce to part of right arm only for collision testing

File: baxter_description/urdf/baxter.urdf (robot description, URDF)
Before this commit: robot baxter, 49 links, 48 joints
Links:
- removed link collision_head_link_1
- removed link collision_head_link_2
- removed link display
- removed link dummyhead1
- removed link head
- removed link head_camera
- removed link left_arm_itb
- removed link left_arm_mount
- removed link left_gripper
- removed link left_gripper_base
- removed link left_hand
- removed link left_hand_accelerometer
- removed link left_hand_camera
- removed link left_hand_camera_axis
- removed link left_hand_range
- removed link left_lower_elbow
- removed link left_lower_forearm
- removed link left_lower_shoulder
- removed link left_torso_itb
- removed link left_upper_elbow
- removed link left_upper_elbow_visual
- removed link left_upper_forearm
- removed link left_upper_forearm_visual
- removed link left_upper_shoulder
- removed link left_wrist
- removed link right_arm_itb
- removed link right_gripper
- removed link right_gripper_base
- removed link right_hand
- removed link right_hand_accelerometer
- removed link right_hand_camera
- removed link right_hand_camera_axis
- removed link right_hand_range
- removed link right_lower_forearm
- removed link right_upper_forearm
- removed link right_upper_forearm_visual
- removed link right_wrist
- removed link screen
- removed link sonar_ring
- added link world
Joints:
- removed joint collision_head_1
- removed joint collision_head_2
- removed joint display_joint
- removed joint dummy
- removed joint head_camera
- removed joint head_nod
- removed joint head_pan
- removed joint left_e0
- removed joint left_e0_fixed
- removed joint left_e1
- removed joint left_endpoint
- removed joint left_gripper_base
- removed joint left_hand
- removed joint left_hand_accelerometer
- removed joint left_hand_camera
- removed joint left_hand_camera_axis
- removed joint left_hand_range
- removed joint left_s0
- removed joint left_s1
- removed joint left_torso_arm_mount
- removed joint left_torso_itb_fixed
- removed joint left_w0
- removed joint left_w0_fixed
- removed joint left_w0_to_itb_fixed
- removed joint left_w1
- removed joint left_w2
- removed joint right_endpoint
- removed joint right_gripper_base
- removed joint right_hand
- removed joint right_hand_accelerometer
- removed joint right_hand_camera
- removed joint right_hand_camera_axis
- removed joint right_hand_range
- removed joint right_w0
- removed joint right_w0_fixed
- removed joint right_w0_to_itb_fixed
- removed joint right_w1
- removed joint right_w2
- removed joint sonar_s0
- added joint fixed: type fixed, parent world, child base
- joint right_s1: limit lower=-2.147 upper=1.047 effort=100.0 velocity=1.5 -> lower=-2.147 upper=1.047 effort=50.0 velocity=1.5

File: baxter_description/urdf/baxter_base/baxter_base.gazebo.xacro (robot description, xacro)
@@ -5,12 +5,48 @@
     <plugin name="baxter_ros_control" filename="libbaxter_gazebo_ros_control.so">
       <robotNamespace>/robot</robotNamespace>
-      <robotSimType>gazebo_ros_control/DefaultRobotHWSim</robotSimType> <!-- Gazebo Default -->
-      <controlPeriod>0.001</controlPeriod> <!-- Gazebo Default -->
+      <robotSimType>gazebo_ros_control/DefaultRobotHWSim</robotSimType>
+      <controlPeriod>0.001</controlPeriod>
     </plugin>
   </gazebo>
   <!-- Gazebo-Specific Link Properties -->
+  <gazebo reference=""> <!-- Whole Model -->
+    <self_collide>true</self_collide>
+  </gazebo>
   <gazebo reference="torso">
     <self_collide>true</self_collide>
   </gazebo>
+  <gazebo reference="pedestal">
+    <self_collide>false</self_collide>
+  </gazebo>
+  <gazebo reference="right_torso_itb">
+    <self_collide>false</self_collide>
+  </gazebo>
+  <gazebo reference="right_arm_mount">
+    <self_collide>false</self_collide>
+  </gazebo>
+  <gazebo reference="right_upper_shoulder">
+    <self_collide>false</self_collide>
+  </gazebo>
+  <gazebo reference="right_lower_shoulder">
+    <self_collide>false</self_collide>
+  </gazebo>
+  <gazebo reference="right_upper_elbow_visual">
+    <self_collide>false</self_collide>
+  </gazebo>
+  <gazebo reference="right_upper_elbow">
+    <self_collide>false</self_collide>
+  </gazebo>
+  <gazebo reference="right_lower_elbow">
+    <self_collide>true</self_collide>
+  </gazebo>
+  <gazebo reference="right_upper_forearm_visual">
+    <self_collide>false</self_collide>
+  </gazebo>
+  <gazebo reference="right_arm_itb">
+    <self_collide>false</self_collide>
+  </gazebo>
+  <gazebo reference="right_lower_forearm">
+    <self_collide>false</self_collide>
+  </gazebo>
   <gazebo reference="head_pan">
     <implicitSpringDamper>1</implicitSpringDamper>
@@ -59,231 +95,231 @@
   </gazebo>
   <!-- Gazebo-Specific Sensor Properties -->
-  <gazebo reference="head_camera">
-    <sensor name="head_camera" type="camera">
-      <update_rate>30.0</update_rate>
-      <camera name="head_camera">
-        <pose>0.0 0.21 0.0 0.0 -0.8 -1.570796327 </pose>
-        <horizontal_fov>1.3962634</horizontal_fov>
-        <image>
-          <width>800</width>
-          <height>800</height>
-          <format>R8G8B8</format>
-        </image>
-        <clip>
-          <near>0.02</near>
-          <far>300</far>
-        </clip>
-        <noise>
-          <type>gaussian</type>
-          <mean>0.0</mean>
-          <stddev>0.007</stddev>
-        </noise>
-      </camera>
-      <plugin filename="libgazebo_ros_camera.so" name="camera_controller">
-        <alwaysOn>true</alwaysOn>
-        <updateRate>0.0</updateRate>
-        <cameraName>head_camera</cameraName>
-        <imageTopicName>image</imageTopicName>
-        <cameraInfoTopicName>camera_info</cameraInfoTopicName>
-        <frameName>head_camera</frameName>
-        <hackBaseline>0.07</hackBaseline>
-        <distortionK1>0.0</distortionK1>
-        <distortionK2>0.0</distortionK2>
-        <distortionK3>0.0</distortionK3>
-        <distortionT1>0.0</distortionT1>
-        <distortionT2>0.0</distortionT2>
-        <CxPrime>0</CxPrime>
-        <Cx>0.0</Cx>
-        <Cy>0.0</Cy>
-        <focalLength>0.0</focalLength>
-        <robotNamespace>/cameras</robotNamespace>
-      </plugin>
-    </sensor>
-  </gazebo>
-  <gazebo reference="right_hand_camera">
-    <sensor name="right_hand_camera" type="camera">
-      <update_rate>30.0</update_rate>
-      <camera name="right_hand_camera">
-        <pose>0.0 0.0 0.0 0.0 -1.570796327 1.570796327 </pose>
-        <horizontal_fov>1.3962634</horizontal_fov>
-        <image>
-          <width>800</width>
-          <height>800</height>
-          <format>R8G8B8</format>
-        </image>
-        <clip>
-          <near>0.02</near>
-          <far>300</far>
-        </clip>
-        <noise>
-          <type>gaussian</type>
-          <mean>0.0</mean>
-          <stddev>0.007</stddev>
-        </noise>
-      </camera>
-      <plugin filename="libgazebo_ros_camera.so" name="camera_controller">
-        <alwaysOn>true</alwaysOn>
-        <updateRate>0.0</updateRate>
-        <cameraName>right_hand_camera</cameraName>
-        <imageTopicName>image</imageTopicName>
-        <cameraInfoTopicName>camera_info</cameraInfoTopicName>
-        <frameName>right_hand_camera</frameName>
-        <hackBaseline>0.07</hackBaseline>
-        <distortionK1>0.0</distortionK1>
-        <distortionK2>0.0</distortionK2>
-        <distortionK3>0.0</distortionK3>
-        <distortionT1>0.0</distortionT1>
-        <distortionT2>0.0</distortionT2>
-        <CxPrime>0</CxPrime>
-        <Cx>0.0</Cx>
-        <Cy>0.0</Cy>
-        <focalLength>0.0</focalLength>
-        <robotNamespace>/cameras</robotNamespace>
-      </plugin>
-    </sensor>
-  </gazebo>
-  <gazebo reference="left_hand_camera">
-    <sensor name="left_hand_camera" type="camera">
-      <update_rate>30.0</update_rate>
-      <camera name="left_hand_camera">
-        <pose>0.0 0.0 0.0 0.0 -1.570796327 1.570796327 </pose>
-        <horizontal_fov>1.3962634</horizontal_fov>
-        <image>
-          <width>800</width>
-          <height>800</height>
-          <format>R8G8B8</format>
-        </image>
-        <clip>
-          <near>0.02</near>
-          <far>300</far>
-        </clip>
-        <noise>
-          <type>gaussian</type>
-          <mean>0.0</mean>
-          <stddev>0.007</stddev>
-        </noise>
-      </camera>
-      <plugin filename="libgazebo_ros_camera.so" name="camera_controller">
-        <alwaysOn>true</alwaysOn>
-        <updateRate>0.0</updateRate>
-        <cameraName>left_hand_camera</cameraName>
-        <imageTopicName>image</imageTopicName>
-        <cameraInfoTopicName>camera_info</cameraInfoTopicName>
-        <frameName>left_hand_camera</frameName>
-        <hackBaseline>0.07</hackBaseline>
-        <distortionK1>0.0</distortionK1>
-        <distortionK2>0.0</distortionK2>
-        <distortionK3>0.0</distortionK3>
-        <distortionT1>0.0</distortionT1>
-        <distortionT2>0.0</distortionT2>
-        <CxPrime>0</CxPrime>
-        <Cx>0.0</Cx>
-        <Cy>0.0</Cy>
-        <focalLength>0.0</focalLength>
-        <robotNamespace>/cameras</robotNamespace>
-      </plugin>
-    </sensor>
-  </gazebo>
-  <gazebo reference="display">
-    <visual>
-      <plugin name="screen_video_controller" filename="libgazebo_ros_video.so">
-        <height>600</height>
-        <width>1024</width>
-        <topicName>/robot/xdisplay</topicName>
-        <robotNamespace>/robot</robotNamespace>
-      </plugin>
-    </visual>
-  </gazebo>
-  <gazebo reference="sonar_ring">
-    <sensor name="sonar" type="ray">
-      <pose>0.0 0.0 0.0 0.0 0.0 0.0</pose>
-      <ray>
-        <scan>
-          <horizontal>
-            <samples>12</samples>
-            <resolution>1.0</resolution>
-            <min_angle>-3.14</min_angle>
-            <max_angle>3.14</max_angle>
-          </horizontal>
-          <vertical>
-            <samples>2</samples>
-            <resolution>1.0</resolution>
-            <min_angle>-0.001</min_angle>
-            <max_angle>0</max_angle>
-          </vertical>
-        </scan>
-        <range>
-          <min>0.05</min>
-          <max>50.0</max>
-        </range>
-      </ray>
-      <plugin name="sonar_plugin" filename="libgazebo_ros_block_laser.so">
-        <gaussianNoise>0.00</gaussianNoise>
-        <alwaysOn>true</alwaysOn>
-        <updateRate>100.0</updateRate>
-        <topicName>/robot/sonar/head_sonar/state</topicName>
-        <frameName>sonar_ring</frameName>
-        <hokuyoMinIntensity>101</hokuyoMinIntensity>
-      </plugin>
-      <always_on>true</always_on>
-      <update_rate>100.0</update_rate>
-    </sensor>
-  </gazebo>
-  <gazebo reference="right_hand_range">
-    <sensor name="ir_right" type="ray">
-      <pose>0.0 0.0 0.0 0.0 0.0 0.0</pose>
-      <ray>
-        <scan>
-          <horizontal>
-            <samples>1</samples>
-            <resolution>1.0</resolution>
-            <min_angle>-0.5</min_angle>
-            <max_angle>0.5</max_angle>
-          </horizontal>
-        </scan>
-        <range>
-          <min>0.004</min>
-          <max>0.4</max>
-        </range>
-      </ray>
-      <plugin name="plugin_3" filename="libgazebo_ros_laser.so">
-        <gaussianNoise>0.005</gaussianNoise>
-        <alwaysOn>true</alwaysOn>
-        <updateRate>100</updateRate>
-        <topicName>/sim/laserscan/right_hand_range/state</topicName>
-        <frameName>right_hand_range</frameName>
-      </plugin>
-      <always_on>true</always_on>
-      <update_rate>100.0</update_rate>
-    </sensor>
-  </gazebo>
-  <gazebo reference="left_hand_range">
-    <sensor name="ir_left" type="ray">
-      <pose>0.0 0.0 0.0 0.0 0.0 0.0</pose>
-      <ray>
-        <scan>
-          <horizontal>
-            <samples>1</samples>
-            <resolution>1.0</resolution>
-            <min_angle>-0.5</min_angle>
-            <max_angle>0.5</max_angle>
-          </horizontal>
-        </scan>
-        <range>
-          <min>0.004</min>
-          <max>0.4</max>
-        </range>
-      </ray>
-      <plugin name="plugin_4" filename="libgazebo_ros_laser.so">
-        <gaussianNoise>0.005</gaussianNoise>
-        <alwaysOn>true</alwaysOn>
-        <updateRate>100</updateRate>
-        <topicName>/sim/laserscan/left_hand_range/state</topicName>
-        <frameName>left_hand_range</frameName>
-      </plugin>
-      <always_on>true</always_on>
-      <update_rate>100.0</update_rate>
-    </sensor>
-  </gazebo>
+  <!-- <gazebo reference="head_camera"> -->
+  <!--   <sensor name="head_camera" type="camera"> -->
+  <!--     <update_rate>30.0</update_rate> -->
+  <!--     <camera name="head_camera"> -->
+  <!--       <pose>0.0 0.21 0.0 0.0 -0.8 -1.570796327 </pose> -->
+  <!--       <horizontal_fov>1.3962634</horizontal_fov> -->
+  <!--       <image> -->
+  <!--         <width>800</width> -->
+  <!--         <height>800</height> -->
+  <!--         <format>R8G8B8</format> -->
+  <!--       </image> -->
+  <!--       <clip> -->
+  <!--         <near>0.02</near> -->
+  <!--         <far>300</far> -->
+  <!--       </clip> -->
+  <!--       <noise> -->
+  <!--         <type>gaussian</type> -->
+  <!--         <mean>0.0</mean> -->
+  <!--         <stddev>0.007</stddev> -->
+  <!--       </noise> -->
+  <!--     </camera> -->
+  <!--     <plugin filename="libgazebo_ros_camera.so" name="camera_controller"> -->
+  <!--       <alwaysOn>true</alwaysOn> -->
+  <!--       <updateRate>0.0</updateRate> -->
+  <!--       <cameraName>head_camera</cameraName> -->
+  <!--       <imageTopicName>image</imageTopicName> -->
+  <!--       <cameraInfoTopicName>camera_info</cameraInfoTopicName> -->
+  <!--       <frameName>head_camera</frameName> -->
+  <!--       <hackBaseline>0.07</hackBaseline> -->
+  <!--       <distortionK1>0.0</distortionK1> -->
+  <!--       <distortionK2>0.0</distortionK2> -->
+  <!--       <distortionK3>0.0</distortionK3> -->
+  <!--       <distortionT1>0.0</distortionT1> -->
+  <!--       <distortionT2>0.0</distortionT2> -->
+  <!--       <CxPrime>0</CxPrime> -->
+  <!--       <Cx>0.0</Cx> -->
+  <!--       <Cy>0.0</Cy> -->
+  <!--       <focalLength>0.0</focalLength> -->
+  <!--       <robotNamespace>/cameras</robotNamespace> -->
+  <!--     </plugin> -->
+  <!--   </sensor> -->
+  <!-- </gazebo> -->
+  <!-- <gazebo reference="right_hand_camera"> -->
+  <!--   <sensor name="right_hand_camera" type="camera"> -->
+  <!--     <update_rate>30.0</update_rate> -->
+  <!--     <camera name="right_hand_camera"> -->
+  <!--       <pose>0.0 0.0 0.0 0.0 -1.570796327 1.570796327 </pose> -->
+  <!--       <horizontal_fov>1.3962634</horizontal_fov> -->
+  <!--       <image> -->
+  <!--         <width>800</width> -->
+  <!--         <height>800</height> -->
+  <!--         <format>R8G8B8</format> -->
+  <!--       </image> -->
+  <!--       <clip> -->
+  <!--         <near>0.02</near> -->
+  <!--         <far>300</far> -->
+  <!--       </clip> -->
+  <!--       <noise> -->
+  <!--         <type>gaussian</type> -->
+  <!--         <mean>0.0</mean> -->
+  <!--         <stddev>0.007</stddev> -->
+  <!--       </noise> -->
+  <!--     </camera> -->
+  <!--     <plugin filename="libgazebo_ros_camera.so" name="camera_controller"> -->
+  <!--       <alwaysOn>true</alwaysOn> -->
+  <!--       <updateRate>0.0</updateRate> -->
+  <!--       <cameraName>right_hand_camera</cameraName> -->
+  <!--       <imageTopicName>image</imageTopicName> -->
+  <!--       <cameraInfoTopicName>camera_info</cameraInfoTopicName> -->
+  <!--       <frameName>right_hand_camera</frameName> -->
+  <!--       <hackBaseline>0.07</hackBaseline> -->
+  <!--       <distortionK1>0.0</distortionK1> -->
+  <!--       <distortionK2>0.0</distortionK2> -->
+  <!--       <distortionK3>0.0</distortionK3> -->
+  <!--       <distortionT1>0.0</distortionT1> -->
+  <!--       <distortionT2>0.0</distortionT2> -->
+  <!--       <CxPrime>0</CxPrime> -->
+  <!--       <Cx>0.0</Cx> -->
+  <!--       <Cy>0.0</Cy> -->
+  <!--       <focalLength>0.0</focalLength> -->
+  <!--       <robotNamespace>/cameras</robotNamespace> -->
+  <!--     </plugin> -->
+  <!--   </sensor> -->
+  <!-- </gazebo> -->
+  <!-- <gazebo reference="left_hand_camera"> -->
+  <!--   <sensor name="left_hand_camera" type="camera"> -->
+  <!--     <update_rate>30.0</update_rate> -->
+  <!--     <camera name="left_hand_camera"> -->
+  <!--       <pose>0.0 0.0 0.0 0.0 -1.570796327 1.570796327 </pose> -->
+  <!--       <horizontal_fov>1.3962634</horizontal_fov> -->
+  <!--       <image> -->
+  <!--         <width>800</width> -->
+  <!--         <height>800</height> -->
+  <!--         <format>R8G8B8</format> -->
+  <!--       </image> -->
+  <!--       <clip> -->
+  <!--         <near>0.02</near> -->
+  <!--         <far>300</far> -->
+  <!--       </clip> -->
+  <!--       <noise> -->
+  <!--         <type>gaussian</type> -->
+  <!--         <mean>0.0</mean> -->
+  <!--         <stddev>0.007</stddev> -->
+  <!--       </noise> -->
+  <!--     </camera> -->
+  <!--     <plugin filename="libgazebo_ros_camera.so" name="camera_controller"> -->
+  <!--       <alwaysOn>true</alwaysOn> -->
+  <!--       <updateRate>0.0</updateRate> -->
+  <!--       <cameraName>left_hand_camera</cameraName> -->
+  <!--       <imageTopicName>image</imageTopicName> -->
+  <!--       <cameraInfoTopicName>camera_info</cameraInfoTopicName> -->
+  <!--       <frameName>left_hand_camera</frameName> -->
+  <!--       <hackBaseline>0.07</hackBaseline> -->
+  <!--       <distortionK1>0.0</distortionK1> -->
+  <!--       <distortionK2>0.0</distortionK2> -->
+  <!--       <distortionK3>0.0</distortionK3> -->
+  <!--       <distortionT1>0.0</distortionT1> -->
+  <!--       <distortionT2>0.0</distortionT2> -->
+  <!--       <CxPrime>0</CxPrime> -->
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