Commit message: Reduce to part of right arm only for collision testing

File: baxter_description/urdf/baxter_base/baxter_base.urdf.xacro (robot description, xacro)
@@ -30,11 +30,11 @@
     </inertial>
   </link>
-  <link name="left_torso_itb">
-    <inertial>
-      <origin rpy="0 0 0" xyz="0.000000 0.000000 0.000000"/>
-      <mass value="0.0001"/>
-      <inertia ixx="1e-08" ixy="0" ixz="0" iyy="1e-08" iyz="0" izz="1e-08"/>
-    </inertial>
-  </link>
+  <!-- <link name="left_torso_itb"> -->
+  <!--   <inertial> -->
+  <!--     <origin rpy="0 0 0" xyz="0.000000 0.000000 0.000000"/> -->
+  <!--     <mass value="0.0001"/> -->
+  <!--     <inertia ixx="1e-08" ixy="0" ixz="0" iyy="1e-08" iyz="0" izz="1e-08"/> -->
+  <!--   </inertial> -->
+  <!-- </link> -->
   <link name="right_torso_itb">
     <inertial>
@@ -44,159 +44,159 @@
     </inertial>
   </link>
-  <link name="head">
-    <visual>
-      <origin rpy="0 0 0" xyz="0 0 .00953"/>
-      <geometry>
-        <mesh filename="package://baxter_description/meshes/head/H0.DAE"/>
-      </geometry>
-      <material name="darkgray">
-        <color rgba=".2 .2 .2 1"/>
-      </material>
-    </visual>
-    <collision>
-      <origin rpy="0 0 0" xyz="0.0 0 0.0"/>
-      <geometry>
-        <sphere radius="0.001"/>
-      </geometry>
-    </collision>
-    <inertial>
-      <origin rpy="0 0 0" xyz="0 0 0"/>
-      <mass value="0.547767"/>
-      <inertia ixx="0.004641" ixy="0.000159" ixz="0.000242" iyy="0.003295" iyz="-0.001324" izz="0.003415"/>
-    </inertial>
-  </link>
-  <link name="sonar_ring">
-    <visual>
-      <origin rpy="0 0 0" xyz="-.0347 0 .00953"/>
-      <geometry>
-        <cylinder length="0.01" radius="0.085"/>
-      </geometry>
-      <material name="darkgray">
-        <color rgba=".2 .2 .2 1"/>
-      </material>
-    </visual>
-    <collision>
-      <origin rpy="0 0 0" xyz="0.0 0 0.0"/>
-      <geometry>
-        <sphere radius="0.001"/>
-      </geometry>
-    </collision>
-    <inertial>
-      <origin rpy="0 0 0" xyz="0 0 0"/>
-      <mass value="0.0001"/>
-      <inertia ixx="1e-08" ixy="0" ixz="0" iyy="1e-08" iyz="0" izz="1e-08"/>
-    </inertial>
-  </link>
-  <link name="screen">
-    <visual>
-      <origin rpy="0 -1.57079632679 0" xyz="0 -.00953 -.0347"/>
-      <geometry>
-        <mesh filename="package://baxter_description/meshes/head/H1.DAE"/>
-      </geometry>
-      <material name="darkred">
-        <color rgba=".5 .1 .1 1"/>
-      </material>
-    </visual>
-    <collision>
-      <origin rpy="0 0 0" xyz="0.0 0 0.0"/>
-      <geometry>
-        <sphere radius="0.001"/>
-      </geometry>
-    </collision>
-    <inertial>
-      <origin rpy="0 0 0" xyz="0 0 0"/>
-      <mass value="0.440171"/>
-      <inertia ixx="0.004006" ixy="0.000230" ixz="0.000002" iyy="0.002800" iyz="0.000029" izz="0.001509"/>
-    </inertial>
-  </link>
-  <link name="display">
-    <visual>
-      <origin rpy="0.2617993877991494 0 0" xyz="0 0 0"/>
-      <geometry>
-        <box size="0.218 0.16 0.001"/>
-      </geometry>
-      <material name="black">
-        <color rgba="0 0 0 1"/>
-      </material>
-    </visual>
-    <inertial>
-      <origin rpy="0 0 0" xyz="0 0 0"/>
-      <mass value="0.0001"/>
-      <inertia ixx="1e-08" ixy="0" ixz="0" iyy="1e-08" iyz="0" izz="1e-08"/>
-    </inertial>
-  </link>
-  <link name="head_camera">
-    <inertial>
-      <origin rpy="0 0 0" xyz="0 0 0"/>
-      <mass value="0.0001"/>
-      <inertia ixx="1e-08" ixy="0" ixz="0" iyy="1e-08" iyz="0" izz="1e-08"/>
-    </inertial>
-  </link>
-  <link name="dummyhead1">
-    <inertial>
-      <origin rpy="0 0 0" xyz="0 0 0"/>
-      <mass value="0.0001"/>
-      <inertia ixx="1e-08" ixy="0" ixz="0" iyy="1e-08" iyz="0" izz="1e-08"/>
-    </inertial>
-  </link>
-  <link name="collision_head_link_1">
-    <visual>
-      <origin rpy="0 0 0" xyz="0 0 0"/>
-      <geometry>
-        <sphere radius="0.001"/>
-      </geometry>
-      <material name="red">
-        <color rgba="0.8 0.3 0.3 0.3"/>
-      </material>
-    </visual>
-    <collision>
-      <origin rpy="0 0 0.0" xyz="-0.07 -0.04 0.0"/>
-      <geometry>
-        <sphere radius="0.22"/>
-      </geometry>
-    </collision>
-    <inertial>
-      <origin rpy="0 0 0" xyz="0 0 0"/>
-      <mass value="0.0001"/>
-      <inertia ixx="1e-08" ixy="0" ixz="0" iyy="1e-08" iyz="0" izz="1e-08"/>
-    </inertial>
-  </link>
-  <link name="collision_head_link_2">
-    <visual>
-      <origin rpy="0 0 0" xyz="0 0 0"/>
-      <geometry>
-        <sphere radius="0.001"/>
-      </geometry>
-      <material name="red">
-        <color rgba="0.8 0.3 0.3 0.3"/>
-      </material>
-    </visual>
-    <collision>
-      <origin rpy="0 0 0" xyz="-0.07 0.04 0.00"/>
-      <geometry>
-        <sphere radius="0.22"/>
-      </geometry>
-    </collision>
-    <inertial>
-      <origin rpy="0 0 0" xyz="0 0 0"/>
-      <mass value="0.0001"/>
-      <inertia ixx="1e-08" ixy="0" ixz="0" iyy="1e-08" iyz="0" izz="1e-08"/>
-    </inertial>
-  </link>
-  <joint name="collision_head_1" type="fixed">
-    <origin rpy="0 0 0" xyz="0.11 0 0.75"/>
-    <parent link="base"/>
-    <child link="collision_head_link_1"/>
-  </joint>
-  <joint name="collision_head_2" type="fixed">
-    <origin rpy="0 0 0" xyz="0.11 0 0.75"/>
-    <parent link="base"/>
-    <child link="collision_head_link_2"/>
-  </joint>
-  <joint name="dummy" type="fixed">
-    <origin rpy="0 0 0" xyz="0 0 0"/>
-    <parent link="head"/>
-    <child link="dummyhead1"/>
-  </joint>
+  <!-- <link name="head"> -->
+  <!--   <visual> -->
+  <!--     <origin rpy="0 0 0" xyz="0 0 .00953"/> -->
+  <!--     <geometry> -->
+  <!--       <mesh filename="package://baxter_description/meshes/head/H0.DAE"/> -->
+  <!--     </geometry> -->
+  <!--     <material name="darkgray"> -->
+  <!--       <color rgba=".2 .2 .2 1"/> -->
+  <!--     </material> -->
+  <!--   </visual> -->
+  <!--   <collision> -->
+  <!--     <origin rpy="0 0 0" xyz="0.0 0 0.0"/> -->
+  <!--     <geometry> -->
+  <!--       <sphere radius="0.001"/> -->
+  <!--     </geometry> -->
+  <!--   </collision> -->
+  <!--   <inertial> -->
+  <!--     <origin rpy="0 0 0" xyz="0 0 0"/> -->
+  <!--     <mass value="0.547767"/> -->
+  <!--     <inertia ixx="0.004641" ixy="0.000159" ixz="0.000242" iyy="0.003295" iyz="-0.001324" izz="0.003415"/> -->
+  <!--   </inertial> -->
+  <!-- </link> -->
+  <!-- <link name="sonar_ring"> -->
+  <!--   <visual> -->
+  <!--     <origin rpy="0 0 0" xyz="-.0347 0 .00953"/> -->
+  <!--     <geometry> -->
+  <!--       <cylinder length="0.01" radius="0.085"/> -->
+  <!--     </geometry> -->
+  <!--     <material name="darkgray"> -->
+  <!--       <color rgba=".2 .2 .2 1"/> -->
+  <!--     </material> -->
+  <!--   </visual> -->
+  <!--   <collision> -->
+  <!--     <origin rpy="0 0 0" xyz="0.0 0 0.0"/> -->
+  <!--     <geometry> -->
+  <!--       <sphere radius="0.001"/> -->
+  <!--     </geometry> -->
+  <!--   </collision> -->
+  <!--   <inertial> -->
+  <!--     <origin rpy="0 0 0" xyz="0 0 0"/> -->
+  <!--     <mass value="0.0001"/> -->
+  <!--     <inertia ixx="1e-08" ixy="0" ixz="0" iyy="1e-08" iyz="0" izz="1e-08"/> -->
+  <!--   </inertial> -->
+  <!-- </link> -->
+  <!-- <link name="screen"> -->
+  <!--   <visual> -->
+  <!--     <origin rpy="0 -1.57079632679 0" xyz="0 -.00953 -.0347"/> -->
+  <!--     <geometry> -->
+  <!--       <mesh filename="package://baxter_description/meshes/head/H1.DAE"/> -->
+  <!--     </geometry> -->
+  <!--     <material name="darkred"> -->
+  <!--       <color rgba=".5 .1 .1 1"/> -->
+  <!--     </material> -->
+  <!--   </visual> -->
+  <!--   <collision> -->
+  <!--     <origin rpy="0 0 0" xyz="0.0 0 0.0"/> -->
+  <!--     <geometry> -->
+  <!--       <sphere radius="0.001"/> -->
+  <!--     </geometry> -->
+  <!--   </collision> -->
+  <!--   <inertial> -->
+  <!--     <origin rpy="0 0 0" xyz="0 0 0"/> -->
+  <!--     <mass value="0.440171"/> -->
+  <!--     <inertia ixx="0.004006" ixy="0.000230" ixz="0.000002" iyy="0.002800" iyz="0.000029" izz="0.001509"/> -->
+  <!--   </inertial> -->
+  <!-- </link> -->
+  <!-- <link name="display"> -->
+  <!--   <visual> -->
+  <!--     <origin rpy="0.2617993877991494 0 0" xyz="0 0 0"/> -->
+  <!--     <geometry> -->
+  <!--       <box size="0.218 0.16 0.001"/> -->
+  <!--     </geometry> -->
+  <!--     <material name="black"> -->
+  <!--       <color rgba="0 0 0 1"/> -->
+  <!--     </material> -->
+  <!--   </visual> -->
+  <!--   <inertial> -->
+  <!--     <origin rpy="0 0 0" xyz="0 0 0"/> -->
+  <!--     <mass value="0.0001"/> -->
+  <!--     <inertia ixx="1e-08" ixy="0" ixz="0" iyy="1e-08" iyz="0" izz="1e-08"/> -->
+  <!--   </inertial> -->
+  <!-- </link> -->
+  <!-- <link name="head_camera"> -->
+  <!--   <inertial> -->
+  <!--     <origin rpy="0 0 0" xyz="0 0 0"/> -->
+  <!--     <mass value="0.0001"/> -->
+  <!--     <inertia ixx="1e-08" ixy="0" ixz="0" iyy="1e-08" iyz="0" izz="1e-08"/> -->
+  <!--   </inertial> -->
+  <!-- </link> -->
+  <!-- <link name="dummyhead1"> -->
+  <!--   <inertial> -->
+  <!--     <origin rpy="0 0 0" xyz="0 0 0"/> -->
+  <!--     <mass value="0.0001"/> -->
+  <!--     <inertia ixx="1e-08" ixy="0" ixz="0" iyy="1e-08" iyz="0" izz="1e-08"/> -->
+  <!--   </inertial> -->
+  <!-- </link> -->
+  <!-- <link name="collision_head_link_1"> -->
+  <!--   <visual> -->
+  <!--     <origin rpy="0 0 0" xyz="0 0 0"/> -->
+  <!--     <geometry> -->
+  <!--       <sphere radius="0.001"/> -->
+  <!--     </geometry> -->
+  <!--     <material name="red"> -->
+  <!--       <color rgba="0.8 0.3 0.3 0.3"/> -->
+  <!--     </material> -->
+  <!--   </visual> -->
+  <!--   <collision> -->
+  <!--     <origin rpy="0 0 0.0" xyz="-0.07 -0.04 0.0"/> -->
+  <!--     <geometry> -->
+  <!--       <sphere radius="0.22"/> -->
+  <!--     </geometry> -->
+  <!--   </collision> -->
+  <!--   <inertial> -->
+  <!--     <origin rpy="0 0 0" xyz="0 0 0"/> -->
+  <!--     <mass value="0.0001"/> -->
+  <!--     <inertia ixx="1e-08" ixy="0" ixz="0" iyy="1e-08" iyz="0" izz="1e-08"/> -->
+  <!--   </inertial> -->
+  <!-- </link> -->
+  <!-- <link name="collision_head_link_2"> -->
+  <!--   <visual> -->
+  <!--     <origin rpy="0 0 0" xyz="0 0 0"/> -->
+  <!--     <geometry> -->
+  <!--       <sphere radius="0.001"/> -->
+  <!--     </geometry> -->
+  <!--     <material name="red"> -->
+  <!--       <color rgba="0.8 0.3 0.3 0.3"/> -->
+  <!--     </material> -->
+  <!--   </visual> -->
+  <!--   <collision> -->
+  <!--     <origin rpy="0 0 0" xyz="-0.07 0.04 0.00"/> -->
+  <!--     <geometry> -->
+  <!--       <sphere radius="0.22"/> -->
+  <!--     </geometry> -->
+  <!--   </collision> -->
+  <!--   <inertial> -->
+  <!--     <origin rpy="0 0 0" xyz="0 0 0"/> -->
+  <!--     <mass value="0.0001"/> -->
+  <!--     <inertia ixx="1e-08" ixy="0" ixz="0" iyy="1e-08" iyz="0" izz="1e-08"/> -->
+  <!--   </inertial> -->
+  <!-- </link> -->
+  <!-- <joint name="collision_head_1" type="fixed"> -->
+  <!--   <origin rpy="0 0 0" xyz="0.11 0 0.75"/> -->
+  <!--   <parent link="base"/> -->
+  <!--   <child link="collision_head_link_1"/> -->
+  <!-- </joint> -->
+  <!-- <joint name="collision_head_2" type="fixed"> -->
+  <!--   <origin rpy="0 0 0" xyz="0.11 0 0.75"/> -->
+  <!--   <parent link="base"/> -->
+  <!--   <child link="collision_head_link_2"/> -->
+  <!-- </joint> -->
+  <!-- <joint name="dummy" type="fixed"> -->
+  <!--   <origin rpy="0 0 0" xyz="0 0 0"/> -->
+  <!--   <parent link="head"/> -->
+  <!--   <child link="dummyhead1"/> -->
+  <!-- </joint> -->
   <joint name="torso_t0" type="fixed">
     <origin rpy="0 0 0" xyz="0 0 0"/>
@@ -205,9 +205,9 @@
     <limit effort="50000" lower="-3.01" upper="3.01" velocity="10000"/>
   </joint>
-  <joint name="left_torso_itb_fixed" type="fixed">
-    <origin rpy="-1.57079632679 3.1415 0" xyz="-0.08897 0.15593 0.389125"/>
-    <parent link="torso"/>
-    <child link="left_torso_itb"/>
-  </joint>
+  <!-- <joint name="left_torso_itb_fixed" type="fixed"> -->
+  <!--   <origin rpy="-1.57079632679 3.1415 0" xyz="-0.08897 0.15593 0.389125"/> -->
+  <!--   <parent link="torso"/> -->
+  <!--   <child link="left_torso_itb"/> -->
+  <!-- </joint> -->
   <joint name="right_torso_itb_fixed" type="fixed">
     <origin rpy="1.57079632679 0 0" xyz="-0.08897 -0.15593 0.389125"/>
@@ -215,33 +215,33 @@
     <child link="right_torso_itb"/>
   </joint>
-  <joint name="head_pan" type="revolute">
-    <origin rpy="0 0 0" xyz="0.06 0 0.686"/>
-    <axis xyz="0 0 1"/>
-    <parent link="torso"/>
-    <child link="head"/>
-    <limit effort="50000" lower="-1.3963" upper="1.3963" velocity="10000"/>
-    <dynamics damping="0.7" friction="0.0"/>
-  </joint>
-  <joint name="head_nod" type="fixed">
-    <origin rpy="1.75057 0 1.57079632679" xyz=".1227 0 0"/>
-    <parent link="head"/>
-    <child link="screen"/>
-  </joint>
-  <joint name="head_camera" type="fixed">
-    <origin rpy="1.75057 0 1.57079632679" xyz="0.12839 0 0.06368"/>
-    <parent link="head"/>
-    <child link="head_camera"/>
-  </joint>
-  <joint name="display_joint" type="fixed">
-    <origin rpy="0 0 0" xyz="0.0 -0.016 0.0"/>
-    <parent link="screen"/>
-    <child link="display"/>
-  </joint>
-  <joint name="sonar_s0" type="fixed">
-    <origin rpy="0 0 0" xyz="0.0947 0 .817"/>
-    <axis xyz="0 0 1"/>
-    <parent link="torso"/>
-    <child link="sonar_ring"/>
-  </joint>
+  <!-- <joint name="head_pan" type="revolute"> -->
+  <!--   <origin rpy="0 0 0" xyz="0.06 0 0.686"/> -->
+  <!--   <axis xyz="0 0 1"/> -->
+  <!--   <parent link="torso"/> -->
+  <!--   <child link="head"/> -->
+  <!--   <limit effort="50000" lower="-1.3963" upper="1.3963" velocity="10000"/> -->
+  <!--   <dynamics damping="0.7" friction="0.0"/> -->
+  <!-- </joint> -->
+  <!-- <joint name="head_nod" type="fixed"> -->
+  <!--   <origin rpy="1.75057 0 1.57079632679" xyz=".1227 0 0"/> -->
+  <!--   <parent link="head"/> -->
+  <!--   <child link="screen"/> -->
+  <!-- </joint> -->
+  <!-- <joint name="head_camera" type="fixed"> -->
+  <!--   <origin rpy="1.75057 0 1.57079632679" xyz="0.12839 0 0.06368"/> -->
+  <!--   <parent link="head"/> -->
+  <!--   <child link="head_camera"/> -->
+  <!-- </joint> -->
+  <!-- <joint name="display_joint" type="fixed"> -->
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